File: Electronics/AberNode/abernode.sch (EAGLE design)
At the start: 11 parts, among them IC1 MCP1703CB, Y2 16MHZ

Commit message: Schematic Mostly Done
Parts:
- added BATT, SOLAR: M02LOCK, SparkFun-Connectors:M02LOCK
- added C6, C9: 10uF, resistor:C-EUC0805
- added C7: (no value), resistor:CPOL-EUE7.5-18
- added CHRG/LBO: ORANGE, led:LEDCHIPLED_0603
- added CON4: (no value), SparkFun-Connectors:M06LONGPADS
- added D1: MBR0520LT, diode:MBR0520LT
- added DONE: GREEN, led:LEDCHIPLED_0603
- added IC2: MCP73871, adafruit:MCP73871
- added PWR: RED, led:LEDCHIPLED_0603
- added R2, R3, R9: 10k, resistor:R-EU_R0805
- added R4: 2K, resistor:R-EU_R0805
- added R5: 100K, resistor:R-EU_R0805
- added R6, R7, R8: 1K, resistor:R-EU_R0805
- added U$1: (no value), tom:ANT
- added U$2, U$3, U$4: HEADER_4, tom:HEADER_4
Connections:
- removed net PSBATT: C1.2, C3.2, IC1.VI
- removed net VCC: C2.2, IC1.VO
- new net ANALOG_1: ATMEGA.(PCINT0/ADC0)PA0, U$2.P$4
- new net ANALOG_2: ATMEGA.(PCINT1/ADC1)PA1, U$3.P$4
- new net ANALOG_3: ATMEGA.(PCINT2/ADC2)PA2, U$4.P$4
- new net ANALOG_4: ATMEGA.(PCINT3/ADC3)PA3, CON4.6
- new net DIGIT_1: ATMEGA.(PCINT24/RXD0)PD0, U$2.P$3
- new net DIGIT_2: ATMEGA.(PCINT25/TXD0)PD1, U$3.P$3
- new net DIGIT_3: ATMEGA.(PCINT26/INT0)PD2, U$4.P$3
- new net N$10: CHRG/LBO.A, R8.1
- new net N$11: IC2./PG, PWR.C
- new net N$12: DONE.C, IC2.STAT2
- new net N$13: CHRG/LBO.C, IC2.STAT1/LBO
- new net N$14: D1.A, SOLAR.2
- new net N$17: IC2.THERM, R9.2
- new net N$5: IC2.PROG3, R5.2
- new net N$6: IC2.VPCC, R2.2, R3.1
- new net N$7: IC2.PROG1, R4.2
- new net N$8: PWR.A, R6.1
- new net N$9: DONE.A, R7.1
- new net SCL: ATMEGA.(PCINT16/SCL)PC0, CON4.5
- new net SDA: ATMEGA.(PCINT17/SDA)PC1, CON4.4
- new net VBATT: BATT.2, C6.2, IC2.VBAT1, IC2.VBAT2, IC2.VBAT3
- new net VIN: C7.+, C9.2, CON4.2, D1.C, IC2./TE, IC2.CE, IC2.IN1, IC2.IN2, IC2.PROG2, IC2.SEL, R3.2, R6.2, R7.2, R8.2
- new net VSUPPLY: C1.2, C3.2, IC1.VI, IC2.OUT1, IC2.OUT2
- net +3V3: now also C2.2, CON4.1, IC1.VO, U$2.P$2, U$3.P$2, U$4.P$2
- net ANT: now also U$1.P$1
- net GND: now also BATT.1, C6.1, C7.-, C9.1, CON4.3, IC2.GND1, IC2.GND2, R2.1, R4.1, R5.1, R9.1, SOLAR.1, U$2.P$1, U$3.P$1, U$4.P$1
- net N$3: now also ATMEGA.AREF
Other:
- note added: "Tom Blanchard"
- moved on the sheet: ATMEGA, C1, C2, C3, C4, C5, FLASH, IC1, R1, Y2

Commit message: Board Designed minus res values
Need to sort out the resistor values for the mcp73871 pullups battery
sense and charging rates.
Parts:
- removed CHRG/LBO: ORANGE, led:LEDCHIPLED_0603
- removed DONE: GREEN, led:LEDCHIPLED_0603
- removed PWR: RED, led:LEDCHIPLED_0603
- added R10, R11: 10k, resistor:R-EU_R0805
Connections:
- removed net N$10: CHRG/LBO.A, R8.1
- removed net N$11: IC2./PG, PWR.C
- removed net N$12: DONE.C, IC2.STAT2
- removed net N$13: CHRG/LBO.C, IC2.STAT1/LBO
- removed net N$8: PWR.A, R6.1
- removed net N$9: DONE.A, R7.1
- new net BATT_SENSE: ATMEGA.(PCINT4/ADC4)PA4, R10.2, R11.1
- new net PG: ATMEGA.(PCINT27/INT1)PD3, IC2./PG, R6.1
- new net STAT1: ATMEGA.(PCINT29/OC1A)PD5, IC2.STAT1/LBO, R8.1
- new net STAT2: ATMEGA.(PCINT28/OC1B)PD4, IC2.STAT2, R7.1
- net GND: now also R10.1
- net VBATT: now also R11.2
Changed lines of the file:
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@@
 <classes>
 <class number="0" name="default" width="0" drill="0">
-<clearance class="0" value="0.205"/>
+<clearance class="0" value="0.2"/>
 </class>
 </classes>
@@
 <part name="R4" library="resistor" deviceset="R-EU_" device="R0805" value="2K"/>
 <part name="R5" library="resistor" deviceset="R-EU_" device="R0805" value="100K"/>
-<part name="PWR" library="led" deviceset="LED" device="CHIPLED_0603" value="RED"/>
-<part name="DONE" library="led" deviceset="LED" device="CHIPLED_0603" value="GREEN"/>
-<part name="CHRG/LBO" library="led" deviceset="LED" device="CHIPLED_0603" value="ORANGE"/>
 <part name="R6" library="resistor" deviceset="R-EU_" device="R0805" value="1K"/>
 <part name="R7" library="resistor" deviceset="R-EU_" device="R0805" value="1K"/>
@@
 <part name="U$3" library="tom" deviceset="HEADER_4" device=""/>
 <part name="U$4" library="tom" deviceset="HEADER_4" device=""/>
+<part name="R10" library="resistor" deviceset="R-EU_" device="R0805" value="10k"/>
+<part name="R11" library="resistor" deviceset="R-EU_" device="R0805" value="10k"/>
+<part name="SUPPLY16" library="supply2" deviceset="GND" device=""/>
 </parts>
 <sheets>
@@
 <instance part="R4" gate="G$1" x="109.22" y="182.88" rot="R90"/>
 <instance part="R5" gate="G$1" x="116.84" y="182.88" rot="R90"/>
-<instance part="PWR" gate="G$1" x="99.06" y="228.6"/>
-<instance part="DONE" gate="G$1" x="88.9" y="228.6"/>
-<instance part="CHRG/LBO" gate="G$1" x="78.74" y="228.6"/>
 <instance part="R6" gate="G$1" x="99.06" y="241.3" rot="R90"/>
 <instance part="R7" gate="G$1" x="88.9" y="241.3" rot="R90"/>
@@
 <instance part="U$3" gate="G$1" x="297.18" y="78.74" rot="R180"/>
 <instance part="U$4" gate="G$1" x="299.72" y="58.42" rot="R180"/>
+<instance part="R10" gate="G$1" x="182.88" y="91.44" rot="R90"/>
+<instance part="R11" gate="G$1" x="182.88" y="104.14" rot="R90"/>
+<instance part="SUPPLY16" gate="GND" x="182.88" y="81.28"/>
 </instances>
 <busses>
@@
 <junction x="290.94" y="73.66"/>
 </segment>
+<segment>
+<pinref part="R10" gate="G$1" pin="1"/>
+<pinref part="SUPPLY16" gate="GND" pin="GND"/>
+<wire x1="182.88" y1="86.36" x2="182.88" y2="83.82" width="0.1524" layer="91"/>
+</segment>
 </net>
 <net name="+3V3" class="0">
@@
 <label x="45.72" y="200.66" size="1.778" layer="95"/>
 </segment>
+<segment>
+<pinref part="R11" gate="G$1" pin="2"/>
+<wire x1="182.88" y1="109.22" x2="198.12" y2="109.22" width="0.1524" layer="91"/>
+<label x="193.04" y="109.22" size="1.778" layer="95"/>
+</segment>
 </net>
 <net name="ANALOG_1" class="0">
@@
 </segment>
 </net>
-<net name="N$8" class="0">
-<segment>
-<pinref part="R6" gate="G$1" pin="1"/>
-<pinref part="PWR" gate="G$1" pin="A"/>
-<wire x1="99.06" y1="236.22" x2="99.06" y2="231.14" width="0.1524" layer="91"/>
-</segment>
-</net>
-<net name="N$9" class="0">
-<segment>
-<pinref part="R7" gate="G$1" pin="1"/>
-<pinref part="DONE" gate="G$1" pin="A"/>
-<wire x1="88.9" y1="236.22" x2="88.9" y2="231.14" width="0.1524" layer="91"/>
-</segment>
-</net>
-<net name="N$10" class="0">
-<segment>
-<pinref part="R8" gate="G$1" pin="1"/>
-<pinref part="CHRG/LBO" gate="G$1" pin="A"/>
-<wire x1="78.74" y1="236.22" x2="78.74" y2="231.14" width="0.1524" layer="91"/>
-</segment>
-</net>
-<net name="N$11" class="0">
-<segment>
-<pinref part="IC2" gate="G$1" pin="/PG"/>
-<pinref part="PWR" gate="G$1" pin="C"/>
-<wire x1="124.46" y1="213.36" x2="99.06" y2="213.36" width="0.1524" layer="91"/>
-<wire x1="99.06" y1="213.36" x2="99.06" y2="223.52" width="0.1524" layer="91"/>
-</segment>
-</net>
-<net name="N$12" class="0">
-<segment>
-<pinref part="IC2" gate="G$1" pin="STAT2"/>
-<pinref part="DONE" gate="G$1" pin="C"/>
-<wire x1="124.46" y1="210.82" x2="88.9" y2="210.82" width="0.1524" layer="91"/>
-<wire x1="88.9" y1="210.82" x2="88.9" y2="223.52" width="0.1524" layer="91"/>
-</segment>
-</net>
-<net name="N$13" class="0">
-<segment>
-<pinref part="IC2" gate="G$1" pin="STAT1/LBO"/>
-<pinref part="CHRG/LBO" gate="G$1" pin="C"/>
-<wire x1="124.46" y1="208.28" x2="78.74" y2="208.28" width="0.1524" layer="91"/>
-<wire x1="78.74" y1="208.28" x2="78.74" y2="223.52" width="0.1524" layer="91"/>
-</segment>
-</net>
 <net name="N$17" class="0">
 <segment>
@@
 </segment>
 </net>
+<net name="PG" class="0">
+<segment>
+<pinref part="ATMEGA" gate="G$1" pin="(PCINT27/INT1)PD3"/>
+<wire x1="119.38" y1="25.4" x2="129.54" y2="25.4" width="0.1524" layer="91"/>
+<label x="124.46" y="25.4" size="1.778" layer="95"/>
+</segment>
+<segment>
+<pinref part="R6" gate="G$1" pin="1"/>
+<pinref part="IC2" gate="G$1" pin="/PG"/>
+<wire x1="124.46" y1="213.36" x2="99.06" y2="213.36" width="0.1524" layer="91"/>
+<wire x1="99.06" y1="213.36" x2="99.06" y2="231.14" width="0.1524" layer="91"/>
+<wire x1="99.06" y1="231.14" x2="99.06" y2="236.22" width="0.1524" layer="91"/>
+<wire x1="99.06" y1="231.14" x2="96.52" y2="231.14" width="0.1524" layer="91"/>
+<wire x1="96.52" y1="231.14" x2="96.52" y2="218.44" width="0.1524" layer="91"/>
+<junction x="99.06" y="231.14"/>
+<label x="96.52" y="220.98" size="1.778" layer="95" rot="R90"/>
+</segment>
+</net>
+<net name="STAT2" class="0">
+<segment>
+<pinref part="ATMEGA" gate="G$1" pin="(PCINT28/OC1B)PD4"/>
+<wire x1="119.38" y1="27.94" x2="129.54" y2="27.94" width="0.1524" layer="91"/>
+<label x="124.46" y="27.94" size="1.778" layer="95"/>
+</segment>
+<segment>
+<pinref part="R7" gate="G$1" pin="1"/>
+<pinref part="IC2" gate="G$1" pin="STAT2"/>
+<wire x1="124.46" y1="210.82" x2="88.9" y2="210.82" width="0.1524" layer="91"/>
+<wire x1="88.9" y1="210.82" x2="88.9" y2="231.14" width="0.1524" layer="91"/>
+<wire x1="88.9" y1="231.14" x2="88.9" y2="236.22" width="0.1524" layer="91"/>
+<wire x1="88.9" y1="231.14" x2="86.36" y2="231.14" width="0.1524" layer="91"/>
+<wire x1="86.36" y1="231.14" x2="86.36" y2="218.44" width="0.1524" layer="91"/>
+<junction x="88.9" y="231.14"/>
+<label x="86.36" y="220.98" size="1.778" layer="95" rot="R90"/>
+</segment>
+</net>
+<net name="STAT1" class="0">
+<segment>
+<pinref part="ATMEGA" gate="G$1" pin="(PCINT29/OC1A)PD5"/>
+<wire x1="119.38" y1="30.48" x2="129.54" y2="30.48" width="0.1524" layer="91"/>
+<label x="124.46" y="30.48" size="1.778" layer="95"/>
+</segment>
+<segment>
+<pinref part="R8" gate="G$1" pin="1"/>
+<pinref part="IC2" gate="G$1" pin="STAT1/LBO"/>
+<wire x1="78.74" y1="236.22" x2="78.74" y2="231.14" width="0.1524" layer="91"/>
+<wire x1="124.46" y1="208.28" x2="78.74" y2="208.28" width="0.1524" layer="91"/>
+<wire x1="78.74" y1="208.28" x2="78.74" y2="231.14" width="0.1524" layer="91"/>
+<wire x1="78.74" y1="231.14" x2="76.2" y2="231.14" width="0.1524" layer="91"/>
+<wire x1="76.2" y1="231.14" x2="76.2" y2="218.44" width="0.1524" layer="91"/>
+<junction x="78.74" y="231.14"/>
+<label x="76.2" y="220.98" size="1.778" layer="95" rot="R90"/>
+</segment>
+</net>
+<net name="BATT_SENSE" class="0">
+<segment>
+<pinref part="R11" gate="G$1" pin="1"/>
+<pinref part="R10" gate="G$1" pin="2"/>
+<wire x1="182.88" y1="99.06" x2="182.88" y2="96.52" width="0.1524" layer="91"/>
+<wire x1="182.88" y1="96.52" x2="167.64" y2="96.52" width="0.1524" layer="91"/>
+<label x="167.64" y="96.52" size="1.778" layer="95"/>
+</segment>
+<segment>
+<pinref part="ATMEGA" gate="G$1" pin="(PCINT4/ADC4)PA4"/>
+<wire x1="119.38" y1="96.52" x2="129.54" y2="96.52" width="0.1524" layer="91"/>
+<label x="124.46" y="96.52" size="1.778" layer="95"/>
+</segment>
+</net>

Commit message: Board redesign
Moved components around, changed orientation of connectors. Added extra
sensor connector. Power to bottom sensor connectors is driven from a
iopin to reduce current draw whilst sleeping.
Parts:
- removed R11: 10k, resistor:R-EU_R0805
- removed RFM: RFM69HW, SparkFun-RF:RFM69HW
- removed U$1: (no value), tom:ANT
- removed U$2: HEADER_4, tom:HEADER_4
- added R12: 10K, resistor:R-EU_R0603
- added RST: (no value), wirepad:SMD2
- added SEN2, SEN3: HEADER_4, tom:HEADER_4
- added U$6: RFM69HW, tom:RFM69HW
- added U$7: (no value), tom:ANT
- C7: value (none) -> 4700u
- R1, R2, R3: value 10k -> 10K; device resistor:R-EU_R0805 -> resistor:R-EU_R0603
- R10, R9: value 10k -> 1M; device resistor:R-EU_R0805 -> resistor:R-EU_R0603
- R4: value 2K -> 4K; device resistor:R-EU_R0805 -> resistor:R-EU_R0603
- R5: device resistor:R-EU_R0805 -> resistor:R-EU_R0603
- R6, R7, R8: value 1K -> 10K; device resistor:R-EU_R0805 -> resistor:R-EU_R0603
- renumbered CON4 to TSEN, U$3 to SEN1, U$4 to SEN4
Connections:
- removed net ANT: RFM.ANT, U$1.P$1
- removed net N$4: ATMEGA.RESET, C5.2, R1.1
- new net ANALOG_5: ATMEGA.(PCINT5/ADC5)PA5, SEN3.P$4
- new net DIGIT_5: ATMEGA.(PCINT30/OC2B/ICP)PD6, SEN3.P$3
- new net N$12: U$6.ANT, U$7.P$1
- new net RESET: ATMEGA.RESET, C5.2, R1.1, RST.P
- new net SENSE_PWR: ATMEGA.(PCINT31/OC2A)PD7, SEN1.P$2, SEN2.P$2, SEN3.P$2, SEN4.P$2
- net +3V3: now also R12.2, R6.2, R7.2, U$6.3.3V; no longer RFM.3.3V, SEN1.P$2, SEN4.P$2, U$2.P$2
- net ANALOG_1: now also SEN2.P$4; no longer U$2.P$4
- net BATT_SENSE: now also R9.1; no longer R11.1
- net DIGIT_1: now also SEN2.P$3; no longer U$2.P$3
- net GND: now also R3.1, R8.1, SEN2.P$1, SEN3.P$1, U$6.GND@1, U$6.GND@2; no longer R2.1, R9.1, RFM.GND@1, RFM.GND@2, U$2.P$1
- net INT_RFM: now also U$6.DIO0; no longer RFM.DIO0
- net MISO: now also U$6.MISO; no longer RFM.MISO
- net MOSI: now also U$6.MOSI; no longer RFM.MOSI
- net N$17: now also R8.2; no longer R9.2
- net N$6: now also R2.1, R3.2; no longer R2.2, R3.1
- net PG: now also R7.1; no longer R6.1
- net SCK: now also U$6.SCK; no longer RFM.SCK
- net SS_RFM: now also U$6.NSS; no longer RFM.NSS
- net STAT1: now also R12.1; no longer R8.1
- net STAT2: now also R6.1; no longer R7.1
- net VBATT: now also R9.2; no longer R11.2
- net VIN: now also R2.2; no longer R3.2, R6.2, R7.2, R8.2
Other:
- moved on the sheet: ATMEGA, R2, R3, R6, R7, R8, R9
