File: Electronics/AberNode/abernode.brd (EAGLE design)
At the start: 39 x 61.9 mm, 35 parts, among them IC1 MCP1703CB, IC2 MCP73871, Y2 16MHZ

Commit message: First Production Version
Parts:
- moved TSEN 1.91 mm to (39.6, 56.3)
Routing:
- net +3V3: track 121.5 -> 162.1 mm
- net ANALOG_4: track 34.9 -> 30.0 mm
- net SCL: track 35.4 -> 31.3 mm
- net VIN: track 100.4 -> 98.9 mm
- net SDA: track 25.7 -> 24.9 mm
Changed lines of the file:
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@@
 </element>
 <element name="D1" library="diode" package="SOD123" value="MBR0520LT" x="39.753" y="4.141" rot="R270"/>
-<element name="TSEN" library="SparkFun-Connectors" package="1X06_LONGPADS" value="" x="39.559" y="58.2" rot="R180"/>
+<element name="TSEN" library="SparkFun-Connectors" package="1X06_LONGPADS" value="" x="39.559" y="56.295" rot="R180"/>
 <element name="SEN2" library="tom" package="HEADER_4" value="HEADER_4" x="16.1918" y="5.129" rot="R180"/>
 <element name="SEN1" library="tom" package="HEADER_4" value="HEADER_4" x="21.5164" y="5.1296" rot="R180"/>
@@
 <wire x1="16.1925" y1="28.2575" x2="16.286" y2="28.531" width="0.254" layer="1"/>
 <wire x1="32.385" y1="34.29" x2="23.1775" y2="34.29" width="0.254" layer="1"/>
-<wire x1="37.465" y1="29.21" x2="33.655" y2="33.02" width="0.254" layer="1"/>
-<wire x1="33.655" y1="33.02" x2="32.385" y2="34.29" width="0.254" layer="1"/>
 <wire x1="23.1775" y1="34.29" x2="22.886" y2="34.331" width="0.254" layer="1"/>
 <wire x1="37.465" y1="29.21" x2="37.771" y2="28.902" width="0.254" layer="1"/>
-<wire x1="9.2075" y1="36.83" x2="7.9375" y2="38.1" width="0.254" layer="16"/>
-<wire x1="9.2075" y1="35.2425" x2="9.2075" y2="36.83" width="0.254" layer="1"/>
-<wire x1="11.1125" y1="35.2425" x2="9.2075" y2="35.2425" width="0.254" layer="1"/>
-<wire x1="7.9375" y1="38.1" x2="7.915" y2="38.134" width="0.254" layer="16"/>
-<wire x1="11.1125" y1="35.2425" x2="11.286" y2="35.131" width="0.254" layer="1"/>
-<wire x1="39.37" y1="33.02" x2="39.37" y2="36.83" width="0.254" layer="1"/>
-<wire x1="39.37" y1="36.83" x2="39.37" y2="58.1025" width="0.254" layer="1"/>
-<wire x1="33.655" y1="33.02" x2="39.37" y2="33.02" width="0.254" layer="1"/>
-<wire x1="39.37" y1="58.1025" x2="39.559" y2="58.2" width="0.254" layer="1"/>
+<wire x1="39.37" y1="33.02" x2="39.37" y2="36.83" width="0.6096" layer="1"/>
 <wire x1="35.2425" y1="36.83" x2="34.925" y2="37.1475" width="0.254" layer="1"/>
 <wire x1="39.37" y1="36.83" x2="35.2425" y2="36.83" width="0.254" layer="1"/>
-<via x="9.2075" y="36.83" extent="1-16" drill="0.3048"/>
 <via x="34.925" y="37.1475" extent="1-16" drill="0.3048"/>
 <wire x1="16.1925" y1="28.2575" x2="16.1925" y2="27.4955" width="0.254" layer="1"/>
@@
 <wire x1="14.097" y1="26.162" x2="14.097" y2="25.488" width="0.254" layer="1"/>
 <wire x1="14.097" y1="25.488" x2="13.97" y2="25.361" width="0.254" layer="1"/>
+<wire x1="37.465" y1="29.21" x2="37.465" y2="31.115" width="0.6096" layer="1"/>
+<wire x1="37.465" y1="31.115" x2="39.37" y2="33.02" width="0.6096" layer="1"/>
+<wire x1="32.385" y1="34.29" x2="32.385" y2="33.02" width="0.254" layer="1"/>
+<wire x1="32.385" y1="33.02" x2="34.036" y2="31.369" width="0.254" layer="1"/>
+<wire x1="34.036" y1="31.369" x2="37.211" y2="31.369" width="0.254" layer="1"/>
+<wire x1="37.211" y1="31.369" x2="37.465" y2="31.115" width="0.254" layer="1"/>
+<wire x1="39.559" y1="56.295" x2="39.559" y2="38.67" width="0.6096" layer="1"/>
+<wire x1="39.559" y1="38.67" x2="39.37" y2="38.481" width="0.6096" layer="1"/>
+<wire x1="39.37" y1="38.481" x2="39.37" y2="36.83" width="0.6096" layer="1"/>
+<wire x1="7.915" y1="38.134" x2="7.915" y2="47.666" width="0.6096" layer="16"/>
+<wire x1="7.915" y1="47.666" x2="10.033" y2="49.784" width="0.6096" layer="16"/>
+<via x="10.033" y="49.784" extent="1-16" drill="0.6" shape="square"/>
+<wire x1="10.033" y1="49.784" x2="10.16" y2="49.784" width="0.6096" layer="1"/>
+<wire x1="10.16" y1="49.784" x2="20.574" y2="60.198" width="0.6096" layer="1"/>
+<wire x1="20.574" y1="60.198" x2="37.592" y2="60.198" width="0.6096" layer="1"/>
+<wire x1="37.592" y1="60.198" x2="39.624" y2="58.166" width="0.6096" layer="1"/>
+<wire x1="39.624" y1="58.166" x2="39.624" y2="56.36" width="0.6096" layer="1"/>
+<wire x1="39.624" y1="56.36" x2="39.559" y2="56.295" width="0.6096" layer="1"/>
 </signal>
 <signal name="N$1">
@@
 <wire x1="11.1125" y1="41.5925" x2="11.1125" y2="29.5275" width="0.254" layer="16"/>
 <wire x1="16.51" y1="46.99" x2="11.1125" y2="41.5925" width="0.254" layer="1"/>
-<wire x1="16.51" y1="55.88" x2="16.51" y2="46.99" width="0.254" layer="1"/>
-<wire x1="21.2725" y1="55.88" x2="16.51" y2="55.88" width="0.254" layer="1"/>
+<wire x1="21.209" y1="46.99" x2="16.51" y2="46.99" width="0.254" layer="1"/>
+<wire x1="21.2725" y1="55.88" x2="21.209" y2="46.99" width="0.254" layer="1"/>
 <wire x1="20.0025" y1="57.15" x2="21.2725" y2="55.88" width="0.254" layer="16"/>
 <wire x1="11.1125" y1="30.1625" x2="11.286" y2="30.331" width="0.254" layer="1"/>
@@
 <wire x1="37.719" y1="17.78" x2="35.441" y2="20.058" width="0.6096" layer="1"/>
 <wire x1="35.441" y1="20.058" x2="34.881" y2="20.058" width="0.6096" layer="1"/>
-<wire x1="40.513" y1="60.833" x2="41.31" y2="60.128" width="0.6096" layer="16"/>
-<wire x1="41.31" y1="60.128" x2="41.31" y2="17.445" width="0.6096" layer="16"/>
+<wire x1="40.64" y1="59.436" x2="41.437" y2="58.731" width="0.6096" layer="16"/>
+<wire x1="41.437" y1="58.731" x2="41.31" y2="17.445" width="0.6096" layer="16"/>
 <wire x1="41.31" y1="17.445" x2="37.91" y2="13.145" width="0.6096" layer="16"/>
 <wire x1="37.91" y1="13.145" x2="37.91" y2="8.844" width="0.6096" layer="16"/>
-<wire x1="37.019" y1="58.2" x2="36.957" y2="58.262" width="0.6096" layer="16"/>
-<wire x1="36.957" y1="58.262" x2="36.957" y2="60.833" width="0.6096" layer="16"/>
-<wire x1="36.957" y1="60.833" x2="40.513" y2="60.833" width="0.6096" layer="16"/>
+<wire x1="37.019" y1="56.295" x2="36.96351875" y2="58.05521875" width="0.6096" layer="16"/>
+<wire x1="36.96351875" y1="58.05521875" x2="37.084" y2="58.135" width="0.6096" layer="16"/>
+<wire x1="40.64" y1="59.436" x2="38.3443" y2="59.436" width="0.6096" layer="16"/>
+<wire x1="38.3443" y1="59.436" x2="36.96351875" y2="58.05521875" width="0.6096" layer="16"/>
 </signal>
 <signal name="N$6">
@@
 <wire x1="28.2575" y1="41.275" x2="23.8125" y2="36.83" width="0.254" layer="1"/>
 <wire x1="28.2575" y1="53.0225" x2="28.2575" y2="41.275" width="0.254" layer="16"/>
-<wire x1="31.75" y1="56.515" x2="28.2575" y2="53.0225" width="0.254" layer="16"/>
-<wire x1="31.75" y1="58.1025" x2="31.75" y2="56.515" width="0.254" layer="16"/>
 <wire x1="23.1775" y1="36.83" x2="22.886" y2="36.731" width="0.254" layer="1"/>
-<wire x1="31.75" y1="58.1025" x2="31.939" y2="58.2" width="0.254" layer="16"/>
 <via x="28.2575" y="41.275" extent="1-16" drill="0.3048"/>
+<wire x1="28.2575" y1="53.0225" x2="30.1625" y2="53.0225" width="0.254" layer="16"/>
+<wire x1="30.1625" y1="53.0225" x2="31.877" y2="54.737" width="0.254" layer="16"/>
+<wire x1="31.877" y1="54.737" x2="31.877" y2="56.233" width="0.254" layer="16"/>
+<wire x1="31.877" y1="56.233" x2="31.939" y2="56.295" width="0.254" layer="16"/>
 </signal>
 <signal name="SCL">
@@
 <wire x1="28.8925" y1="35.8775" x2="23.1775" y2="35.8775" width="0.254" layer="1"/>
 <wire x1="34.925" y1="41.91" x2="28.8925" y2="35.8775" width="0.254" layer="1"/>
-<wire x1="34.925" y1="55.88" x2="34.925" y2="41.91" width="0.254" layer="1"/>
-<wire x1="31.4325" y1="55.88" x2="34.925" y2="55.88" width="0.254" layer="1"/>
-<wire x1="29.21" y1="58.1025" x2="31.4325" y2="55.88" width="0.254" layer="1"/>
 <wire x1="23.1775" y1="35.8775" x2="22.886" y2="35.931" width="0.254" layer="1"/>
-<wire x1="29.21" y1="58.1025" x2="29.399" y2="58.2" width="0.254" layer="1"/>
+<wire x1="34.925" y1="41.91" x2="34.925" y2="44.831" width="0.254" layer="1"/>
+<wire x1="34.925" y1="44.831" x2="29.337" y2="50.419" width="0.254" layer="1"/>
+<wire x1="29.337" y1="50.419" x2="29.337" y2="56.233" width="0.254" layer="1"/>
+<wire x1="29.337" y1="56.233" x2="29.399" y2="56.295" width="0.254" layer="1"/>
 </signal>
 <signal name="N$5">
@@
 <wire x1="12.3825" y1="39.0525" x2="12.065" y2="39.0525" width="0.254" layer="1"/>
 <wire x1="12.3825" y1="43.815" x2="12.3825" y2="39.0525" width="0.254" layer="16"/>
-<wire x1="12.3825" y1="58.1025" x2="12.3825" y2="43.815" width="0.254" layer="1"/>
-<wire x1="26.67" y1="58.1025" x2="12.3825" y2="58.1025" width="0.254" layer="1"/>
 <wire x1="11.43" y1="38.4175" x2="11.286" y2="38.331" width="0.254" layer="1"/>
-<wire x1="26.67" y1="58.1025" x2="26.859" y2="58.2" width="0.254" layer="1"/>
 <via x="12.3825" y="39.0525" extent="1-16" drill="0.3048"/>
 <via x="12.3825" y="43.815" extent="1-16" drill="0.3048"/>
+<wire x1="22.0345" y1="58.1025" x2="19.431" y2="55.499" width="0.254" layer="1"/>
+<wire x1="19.431" y1="55.499" x2="19.431" y2="50.8635" width="0.254" layer="1"/>
+<wire x1="19.431" y1="50.8635" x2="12.3825" y2="43.815" width="0.254" layer="1"/>
+<wire x1="22.0345" y1="58.1025" x2="25.0515" y2="58.1025" width="0.254" layer="1"/>
+<wire x1="25.0515" y1="58.1025" x2="26.859" y2="56.295" width="0.254" layer="1"/>
 </signal>
 <signal name="PG">
@@
 <wire x1="15.5575" y1="28.2575" x2="15.486" y2="28.531" width="0.254" layer="1"/>
 <wire x1="13.0175" y1="23.8125" x2="13.0175" y2="23.878" width="0.254" layer="1"/>
-<wire x1="8.89" y1="33.3375" x2="8.001" y2="33.3375" width="0.254" layer="16"/>
+<wire x1="8.89" y1="33.3375" x2="6.731" y2="33.3375" width="0.254" layer="16"/>
 <wire x1="8.89" y1="26.3525" x2="8.89" y2="33.3375" width="0.254" layer="1"/>
 <wire x1="13.335" y1="26.3525" x2="8.89" y2="26.3525" width="0.254" layer="1"/>
-<wire x1="8.001" y1="33.3375" x2="6.098" y2="33.404" width="0.254" layer="16"/>
+<wire x1="6.731" y1="33.3375" x2="6.098" y2="33.404" width="0.254" layer="16"/>
 <via x="8.89" y="33.3375" extent="1-16" drill="0.3048"/>
 <wire x1="15.5575" y1="28.2575" x2="15.5575" y2="27.6225" width="0.254" layer="1"/>
